Commit message: robot localisation

File: bot_real_description/urdf/bot_real.urdf (robot description, URDF)
Before this commit: robot bot, 7 links, 6 joints
Links:
- link LBW_link: geometry collision cylinder length=0.055 radius=0.065; visual cylinder length=0.055 radius=0.065
- link LFW_link: geometry collision cylinder length=0.055 radius=0.065; visual cylinder length=0.055 radius=0.065
- link RBW_link: geometry collision cylinder length=0.055 radius=0.065; visual cylinder length=0.055 radius=0.065
- link RFW_link: geometry collision cylinder length=0.055 radius=0.065; visual cylinder length=0.055 radius=0.065

Commit message: IMU readings fixed

File: bot_real_description/urdf/bot_real.urdf (robot description, URDF)
Before this commit: robot bot, 7 links, 6 joints
Links:
- added link gps_link, mass 0.001; collision box size=0.001 0.001 0.001; visual box size=0.001 0.001 0.001
Joints:
- added joint gps_joint: type fixed, parent base_link, child gps_link, origin xyz=0.05 0.0 0.1 rpy=0.0 0.0 0.0

Commit message: bot_controller package for joint velocity controller

File: bot_real_description/urdf/bot_real.urdf (robot description, URDF)
Before this commit: robot bot, 7 links, 6 joints
Links:
- added link gps_link, mass 0.001; collision box size=0.001 0.001 0.001; visual box size=0.001 0.001 0.001
Joints:
- added joint gps_joint: type fixed, parent base_link, child gps_link, origin xyz=0.05 0.0 0.1 rpy=0.0 0.0 0.0
- joint LBW_joint: limit effort=100 velocity=100 -> (none)
- joint LFW_joint: limit effort=100 velocity=100 -> (none)
- joint RBW_joint: limit effort=100 velocity=100 -> (none)
- joint RFW_joint: limit effort=100 velocity=100 -> (none)
