Commit message: up and running

File: bot_description/urdf/bot.urdf (robot description, URDF)
Before this commit: robot bot, 7 links, 6 joints
Joints:
- removed joint base_footprint_joint
- added joint base_joint: type fixed, parent base_footprint, child base_link, origin xyz=0.0 0.0 0.0 rpy=0.0 0.0 1.5707

Commit message: upgraded urdf

File: bot_description/urdf/bot.urdf (robot description, URDF)
Before this commit: robot bot, 7 links, 6 joints
Joints:
- joint LBW_joint: axis 1.0 0.0 0.0 -> 0.0 1.0 0.0; child LBW_link -> LFW_link; origin xyz=-0.137 -0.0975 0.0 rpy=0.0 0.0 0.0 -> xyz= -0.0975 0.130 0.0 rpy=0.0 0.0 0.0
- joint LFW_joint: axis 1.0 0.0 0.0 -> 0.0 1.0 0.0; child LFW_link -> RFW_link; origin xyz=-0.137 0.0975 0.0 rpy=0.0 0.0 0.0 -> xyz= 0.0975 0.130 0.0 rpy=0.0 0.0 0.0
- joint RBW_joint: axis 1.0 0.0 0.0 -> 0.0 1.0 0.0; origin xyz=0.130 -0.0975 0.0 rpy=0.0 0.0 0.0 -> xyz=-0.0975 -0.137 0.0 rpy=0.0 0.0 0.0
- joint RFW_joint: axis 1.0 0.0 0.0 -> 0.0 1.0 0.0; child RFW_link -> LBW_link; origin xyz=0.130 0.0975 0.0 rpy=0.0 0.0 0.0 -> xyz=0.0975 -0.137  0.0 rpy=0.0 0.0 0.0
- joint base_joint: origin xyz=0.0 0.0 0.0 rpy=0.0 0.0 1.5707 -> xyz=0.0 0.0 0.0 rpy=0.0 0.0 0

File: bot_real_description/urdf/bot_real.urdf (robot description, URDF)
Before this commit: robot bot, 7 links, 6 joints
Joints:
- joint LBW_joint: axis 1.0 0.0 0.0 -> 0.0 1.0 0.0; child LBW_link -> LFW_link; origin xyz=-0.137 -0.0975 0.0 rpy=0.0 0.0 0.0 -> xyz= -0.0975 0.130 0.0 rpy=0.0 0.0 0.0
- joint LFW_joint: axis 1.0 0.0 0.0 -> 0.0 1.0 0.0; child LFW_link -> RFW_link; origin xyz=-0.137 0.0975 0.0 rpy=0.0 0.0 0.0 -> xyz= 0.0975 0.130 0.0 rpy=0.0 0.0 0.0
- joint RBW_joint: axis 1.0 0.0 0.0 -> 0.0 1.0 0.0; origin xyz=0.130 -0.0975 0.0 rpy=0.0 0.0 0.0 -> xyz=-0.0975 -0.137 0.0 rpy=0.0 0.0 0.0
- joint RFW_joint: axis 1.0 0.0 0.0 -> 0.0 1.0 0.0; child RFW_link -> LBW_link; origin xyz=0.130 0.0975 0.0 rpy=0.0 0.0 0.0 -> xyz=0.0975 -0.137  0.0 rpy=0.0 0.0 0.0
- joint base_joint: origin xyz=0.0 0.0 0.0 rpy=0.0 0.0 1.5707 -> xyz=0.0 0.0 0.0 rpy=0.0 0.0 0

Commit message: Gps readings fixed

File: bot_description/urdf/bot.urdf (robot description, URDF)
Before this commit: robot bot, 7 links, 6 joints
Links:
- added link imu_link, mass 0.001; collision box size=0.001 0.001 0.001; visual box size=0.001 0.001 0.001
Joints:
- added joint imu_joint: type fixed, parent base_link, child imu_link, origin xyz=0.0 0.0 0.1 rpy=0.0 0.0 0.0
- joint LBW_joint: axis 1.0 0.0 0.0 -> 0.0 1.0 0.0; child LBW_link -> LFW_link; origin xyz=-0.137 -0.0975 0.0 rpy=0.0 0.0 0.0 -> xyz= -0.0975 0.130 0.0 rpy=0.0 0.0 0.0
- joint LFW_joint: axis 1.0 0.0 0.0 -> 0.0 1.0 0.0; child LFW_link -> RFW_link; origin xyz=-0.137 0.0975 0.0 rpy=0.0 0.0 0.0 -> xyz= 0.0975 0.130 0.0 rpy=0.0 0.0 0.0
- joint RBW_joint: axis 1.0 0.0 0.0 -> 0.0 1.0 0.0; origin xyz=0.130 -0.0975 0.0 rpy=0.0 0.0 0.0 -> xyz=-0.0975 -0.137 0.0 rpy=0.0 0.0 0.0
- joint RFW_joint: axis 1.0 0.0 0.0 -> 0.0 1.0 0.0; child RFW_link -> LBW_link; origin xyz=0.130 0.0975 0.0 rpy=0.0 0.0 0.0 -> xyz=0.0975 -0.137  0.0 rpy=0.0 0.0 0.0
- joint base_joint: origin xyz=0.0 0.0 0.0 rpy=0.0 0.0 1.5707 -> xyz=0.0 0.0 0.0 rpy=0.0 0.0 0
- joint gps_joint: origin xyz=0.0 0.0 0.1 rpy=0.0 0.0 0.0 -> xyz=0.05 0.0 0.1 rpy=0.0 0.0 0.0

File: bot_description/urdf/bot_real.urdf (robot description, URDF)
Before this commit: robot bot, 7 links, 6 joints
Links:
- link LBW_link: geometry collision mesh filename=package://bot_description/models/meshes/roue.dae; visual mesh filename=package://bot_description/models/meshes/roue.dae
- link LFW_link: geometry collision mesh filename=package://bot_description/models/meshes/roue.dae; visual mesh filename=package://bot_description/models/meshes/roue.dae
- link RBW_link: geometry collision mesh filename=package://bot_description/models/meshes/roue.dae; visual mesh filename=package://bot_description/models/meshes/roue.dae
- link RFW_link: geometry collision mesh filename=package://bot_description/models/meshes/roue.dae; visual mesh filename=package://bot_description/models/meshes/roue.dae
Joints:
- joint LBW_joint: axis 0.0 1.0 0.0 -> 1.0 0.0 0.0; child LFW_link -> LBW_link; origin xyz= -0.0975 0.130 0.0 rpy=0.0 0.0 0.0 -> xyz=-0.137 -0.0975 0.0 rpy=0.0 0.0 0.0
- joint LFW_joint: axis 0.0 1.0 0.0 -> 1.0 0.0 0.0; child RFW_link -> LFW_link; origin xyz= 0.0975 0.130 0.0 rpy=0.0 0.0 0.0 -> xyz=-0.137 0.0975 0.0 rpy=0.0 0.0 0.0
- joint RBW_joint: axis 0.0 1.0 0.0 -> 1.0 0.0 0.0; origin xyz=-0.0975 -0.137 0.0 rpy=0.0 0.0 0.0 -> xyz=0.130 -0.0975 0.0 rpy=0.0 0.0 0.0
- joint RFW_joint: axis 0.0 1.0 0.0 -> 1.0 0.0 0.0; child LBW_link -> RFW_link; origin xyz=0.0975 -0.137  0.0 rpy=0.0 0.0 0.0 -> xyz=0.130 0.0975 0.0 rpy=0.0 0.0 0.0
- joint base_joint: origin xyz=0.0 0.0 0.0 rpy=0.0 0.0 0 -> xyz=0.0 0.0 0.0 rpy=0.0 0.0 1.5707

Commit message: added outdoor navigation package

File: bot_description/urdf/bot.urdf (robot description, URDF)
Before this commit: robot bot, 8 links, 7 joints
Joints:
- joint LBW_joint: limit effort=100 velocity=100 -> effort=100 velocity=30
- joint LFW_joint: limit effort=100 velocity=100 -> effort=100 velocity=30
- joint RBW_joint: limit effort=100 velocity=100 -> effort=100 velocity=30
- joint RFW_joint: limit effort=100 velocity=100 -> effort=100 velocity=30
