Commit message: reset all files and clean

File: bot_simulation/bot_description/urdf/bot.urdf (robot description, URDF)
Before this commit: robot bot, 8 links, 7 joints
Links:
- removed link gps
- added link gps_link, mass 0.001; collision box size=0.001 0.001 0.001; visual box size=0.001 0.001 0.001
- link LBW_link: geometry collision mesh filename=package://bot_description/models/meshes/roue.dae; visual mesh filename=package://bot_description/models/meshes/roue.dae
- link LFW_link: geometry collision mesh filename=package://bot_description/models/meshes/roue.dae; visual mesh filename=package://bot_description/models/meshes/roue.dae
- link RBW_link: geometry collision mesh filename=package://bot_description/models/meshes/roue.dae; visual mesh filename=package://bot_description/models/meshes/roue.dae
- link RFW_link: geometry collision mesh filename=package://bot_description/models/meshes/roue.dae; visual mesh filename=package://bot_description/models/meshes/roue.dae
Joints:
- joint LBW_joint: limit effort=100 velocity=100 -> effort=100 velocity=30
- joint LFW_joint: limit effort=100 velocity=100 -> effort=100 velocity=30
- joint RBW_joint: limit effort=100 velocity=100 -> effort=100 velocity=30
- joint RFW_joint: limit effort=100 velocity=100 -> effort=100 velocity=30
- joint gps_joint: child gps -> gps_link

Commit message: usual testing

File: bot_simulation/bot_description/urdf/bot.urdf (robot description, URDF)
Before this commit: robot bot, 8 links, 7 joints
Links:
- link LBW_link: geometry collision cylinder length=0.055 radius=0.065; visual cylinder length=0.055 radius=0.065
- link LFW_link: geometry collision cylinder length=0.055 radius=0.065; visual cylinder length=0.055 radius=0.065
- link RBW_link: geometry collision cylinder length=0.055 radius=0.065; visual cylinder length=0.055 radius=0.065
- link RFW_link: geometry collision cylinder length=0.055 radius=0.065; visual cylinder length=0.055 radius=0.065
- link gps_link: geometry collision box size=0.01 0.01 0.01; visual box size=0.01 0.01 0.01
- link imu_link: geometry collision box size=0.01 0.01 0.01; visual box size=0.01 0.01 0.01
Joints:
- joint gps_joint: origin xyz=0.05 0.0 0.1 rpy=0.0 0.0 0.0 -> xyz=0.095 0.0 0.245 rpy=0.0 0.0 0.0
- joint imu_joint: origin xyz=0.0 0.0 0.1 rpy=0.0 0.0 0.0 -> xyz=-0.1 0.0 0.245 rpy=0.0 0.0 0.0
