Commit message: move base works on real bot

File: jetson/bot_real/bot_real_description/urdf/bot_real.urdf (robot description, URDF)
Before this commit: robot bot, 8 links, 7 joints
Links:
- added link fake_laser_link
Joints:
- added joint fake_laser_joint: type fixed, parent base_link, child fake_laser_link, origin xyz=0.0 0.0 0.0 rpy=0.0 0.0 0
- joint gps_joint: origin xyz=0.05 0.0 0.1 rpy=0.0 0.0 0.0 -> xyz=0.095 0.0 0.245 rpy=0.0 0.0 0.0
- joint imu_joint: origin xyz=0.0 0.0 0.1 rpy=0.0 0.0 0.0 -> xyz=-0.1 0.0 0.245 rpy=0.0 0.0 3.14

File: jetson/bot_simulation/bot_description/urdf/bot.urdf (robot description, URDF)
Before this commit: robot bot, 8 links, 7 joints
Links:
- added link fake_laser_link
Joints:
- added joint fake_laser_joint: type fixed, parent base_link, child fake_laser_link, origin xyz=0.0 0.0 0.0 rpy=0.0 0.0 0

Commit message: last version

File: jetson/bot_real/bot_real_description/urdf/bot_real.urdf (robot description, URDF)
Before this commit: robot bot, 9 links, 8 joints
Joints:
- joint imu_joint: origin xyz=-0.1 0.0 0.245 rpy=0.0 0.0 3.14 -> xyz=-0.1 0.0 0.245 rpy=0.0 0.0 -1.5707

Commit message: new urdf

File: jetson/bot_real/bot_real_description/urdf/bot_real.urdf (robot description, URDF)
Before this commit: robot bot, 9 links, 8 joints
Links:
- link LBW_link: geometry collision cylinder length=0.025 radius=0.0325; visual cylinder length=0.025 radius=0.0325
- link LFW_link: geometry collision cylinder length=0.025 radius=0.0325; visual cylinder length=0.025 radius=0.0325
- link RBW_link: geometry collision cylinder length=0.025 radius=0.0325; visual cylinder length=0.025 radius=0.0325
- link RFW_link: geometry collision cylinder length=0.025 radius=0.0325; visual cylinder length=0.025 radius=0.0325
- link base_link: geometry collision box size=0.25 0.2 0.16; visual box size=0.25 0.2 0.16
- link gps_link: geometry collision box size=0.03 0.03 0.02; visual box size=0.03 0.03 0.02
- link imu_link: geometry collision box size=0.04 0.07 0.015; visual box size=0.04 0.07 0.015
Joints:
- joint LBW_joint: origin xyz= -0.0975 0.130 0.0 rpy=0.0 0.0 0.0 -> xyz= -0.0575 0.115 0.0 rpy=0.0 0.0 0.0
- joint LFW_joint: origin xyz= 0.0975 0.130 0.0 rpy=0.0 0.0 0.0 -> xyz= 0.0575 0.115 0.0 rpy=0.0 0.0 0.0
- joint RBW_joint: origin xyz=-0.0975 -0.137 0.0 rpy=0.0 0.0 0.0 -> xyz=-0.0575 -0.115 0.0 rpy=0.0 0.0 0.0
- joint RFW_joint: origin xyz=0.0975 -0.137  0.0 rpy=0.0 0.0 0.0 -> xyz=0.0575 -0.115  0.0 rpy=0.0 0.0 0.0
- joint gps_joint: origin xyz=0.095 0.0 0.245 rpy=0.0 0.0 0.0 -> xyz=0.095 0.0 0.18 rpy=0.0 0.0 0.0
- joint imu_joint: origin xyz=-0.1 0.0 0.245 rpy=0.0 0.0 3.14 -> xyz=-0.07 0.0 0.18 rpy=0.0 0.0 3.14

Commit message: urdf gps accurate

File: jetson/bot_real/bot_real_description/urdf/bot_real.urdf (robot description, URDF)
Before this commit: robot bot, 9 links, 8 joints
Links:
- link imu_link: geometry collision box size=0.01 0.02 0.015; visual box size=0.01 0.02 0.015
Joints:
- joint gps_joint: origin xyz=0.095 0.0 0.18 rpy=0.0 0.0 0.0 -> xyz=0.07 0.0 0.18 rpy=0.0 0.0 0.0
- joint imu_joint: origin xyz=-0.07 0.0 0.18 rpy=0.0 0.0 3.14 -> xyz=-0.05 0.0 0.18 rpy=0.0 0.0 3.14
